File: so_26_test_pcb/so_26_test_pcb.kicad_sch (KiCad schematic)
At the start: 0 parts

Commit message: schematic: updated title block
Other:
- company: (none) -> Armin Jahanshahi
- title: (none) -> so_26_test_pcb
Changed lines of the file:
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@@
 	(generator_version "9.0")
 	(paper "A4")
+	(title_block
+		(title "so_26_test_pcb")
+		(date "2026-01-28")
+		(rev "1")
+		(company "Armin Jahanshahi")
+	)
 	(sheet_instances
 		(path "/"
